File: 03_Conception_PCB/Nœud capteur IIoT ultra-basse conso_LoRaWAN & energy harvesting/PCB_deisgn/_autosave-PCB_deisgn.kicad_sch (KiCad schematic)
At the start: 24 parts, among them J1 SWD1, U1 AEM10941-QFN, U2 STM32U073C8Ux, Y1 Crystal

Commit message: feat(sch): add STM32U073 mcu symbol and power pins feat(sch): add mcu decoupling and VDDA ferrite filter feat(sch): add NRST reset and BOOT0 config
feat(sch): add STM32U073 mcu symbol and power pins
feat(sch): add mcu decoupling and VDDA ferrite filter
feat(sch): add NRST reset and BOOT0 config
Parts:
- C13, C14: value 10 µF -> 10 pF
Connections:
- no-connect marks 15 -> 49
